File: Canna/Canna.kicad_pcb (KiCad board)
At the start: 2 copper layers, 70.7 x 53.3 mm, 13 parts, among them J1 NEIGHBOR1, J2 NEIGHBOR2, J7 BONUS_ROW, U1 M24C02-FMN6TP

Commit message: Finish rev1
Parts:
- added C2: 100nF, Capacitor_SMD:C_0603_1608Metric_Pad1.05x0.95mm_HandSolder, F.Cu at (152.7, 101.3)
- added C3: 47nF, Capacitor_SMD:C_0603_1608Metric_Pad1.05x0.95mm_HandSolder, F.Cu at (131.1, 92.9)
- added C4: 100pF, Capacitor_SMD:C_0603_1608Metric_Pad1.05x0.95mm_HandSolder, F.Cu at (122.5, 107.9)
- added C5: 100pF, Capacitor_SMD:C_0603_1608Metric_Pad1.05x0.95mm_HandSolder, F.Cu at (125.9, 92.9)
- added C6: 100pF, Capacitor_SMD:C_0603_1608Metric_Pad1.05x0.95mm_HandSolder, F.Cu at (163.3, 90.8)
- added C7: 100pF, Capacitor_SMD:C_0603_1608Metric_Pad1.05x0.95mm_HandSolder, F.Cu at (159.7, 103.7)
- added C8: 47nF, Capacitor_SMD:C_0603_1608Metric_Pad1.05x0.95mm_HandSolder, F.Cu at (156.3, 103.7)
- added C9: 100nF, Capacitor_SMD:C_0603_1608Metric_Pad1.05x0.95mm_HandSolder, F.Cu at (132.2, 97.5)
- added J3: Screw_Terminal_01x03, TerminalBlock_Phoenix:TerminalBlock_Phoenix_MKDS-1,5-3-5.08_1x03_P5.08mm_Horizontal, F.Cu at (116.0, 102.3)
- added J4: Screw_Terminal_01x03, TerminalBlock_Phoenix:TerminalBlock_Phoenix_MKDS-1,5-3-5.08_1x03_P5.08mm_Horizontal, F.Cu at (170.9, 91.7)
- added JP4: Jumper_2_Bridged, Connector_PinHeader_2.54mm:PinHeader_1x02_P2.54mm_Vertical, F.Cu at (125.9, 97.9)
- added JP5: Jumper_2_Bridged, Connector_PinHeader_2.54mm:PinHeader_1x02_P2.54mm_Vertical, F.Cu at (159.8, 99.4)
- added R2: 120Ohm, Resistor_SMD:R_0603_1608Metric_Pad1.05x0.95mm_HandSolder, F.Cu at (125.9, 106.1)
- added R3: 120Ohm, Resistor_SMD:R_0603_1608Metric_Pad1.05x0.95mm_HandSolder, F.Cu at (159.8, 92.7)
- added U2: TJA1042T-3, Package_SO:SOIC-8_3.9x4.9mm_P1.27mm, F.Cu at (134.0, 101.7)
- added U3: TJA1042T-3, Package_SO:SOIC-8_3.9x4.9mm_P1.27mm, F.Cu at (150.8, 96.5)
Routing:
- net +5V: track 0.00 -> 66.7 mm
- net /P1_18: track 0.00 -> 39.8 mm
- net GND: track 8.65 -> 46.4 mm, vias 3 -> 7
- net /P3_1: track 0.00 -> 29.2 mm
- net /P1_17: track 0.00 -> 28.8 mm
- net /P3_2: track 0.00 -> 24.7 mm
- net /CANL0: track 0.00 -> 22.9 mm
- net /CANL1: track 0.00 -> 20.9 mm
- net /CANH1: track 0.00 -> 19.2 mm
- net /CANH0: track 0.00 -> 19.1 mm
- net /P2_11: track 0.00 -> 18.9 mm
- net /P1_0: track 0.00 -> 16.5 mm
- net VCC: track 29.9 -> 42.3 mm
- net Net-(JP4-Pad2): track 0.00 -> 4.82 mm
- net Net-(JP5-Pad2): track 0.00 -> 3.24 mm
Other:
- board text added: "27 November 2019"
- board text added: "Canna rev1"
- board text added: "JLCJLCJLCJLC"
- board text removed: "24 September 2019"
- board text removed: "My Neighbor"

Commit message: Update rev1 for fab
Other:
- board text added: "CANH0"
- board text added: "CANH1"
- board text added: "CANL0"
- board text added: "CANL1"
Changed lines of the file:
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@@
   (general
     (thickness 1.6)
-    (drawings 236)
+    (drawings 242)
     (tracks 194)
     (zones 0)
@@
     (44 Edge.Cuts user)
     (45 Margin user)
-    (46 B.CrtYd user)
+    (46 B.CrtYd user hide)
     (47 F.CrtYd user)
     (48 B.Fab user)
-    (49 F.Fab user)
+    (49 F.Fab user hide)
   )
   (setup
-    (last_trace_width 0.3048)
+    (last_trace_width 0.2032)
     (user_trace_width 0.3048)
     (user_trace_width 0.508)
@@
   (module neighbor:0603-JUMPER-3-BRIDGED12 (layer F.Cu)
     (at 157.05 82.25)
+    (attr smd)
     (fp_text reference JP2 (at -2.9 0) (layer F.SilkS)
       (effects (font (size 0.6096 0.6096) (thickness 0.1524)))
@@
   (module neighbor:0603-JUMPER-3-BRIDGED12 (layer F.Cu)
     (at 157.05 84.25)
+    (attr smd)
     (fp_text reference JP3 (at -2.9 0) (layer F.SilkS)
       (effects (font (size 0.6096 0.6096) (thickness 0.1524)))
@@
   (module neighbor:0603-JUMPER-3-BRIDGED12 (layer F.Cu)
     (at 157.05 80.25)
+    (attr smd)
     (fp_text reference JP1 (at -2.9 0) (layer F.SilkS)
       (effects (font (size 0.6096 0.6096) (thickness 0.1524)))
@@
     (tags "capacitor handsolder")
     (attr smd)
-    (fp_text reference C6 (at 0 -1.43 270) (layer F.SilkS)
+    (fp_text reference C6 (at -1.94 1.63 270) (layer F.SilkS)
       (effects (font (size 1 1) (thickness 0.15)))
     )
@@
     (tags "resistor handsolder")
     (attr smd)
-    (fp_text reference R3 (at 0 -1.43 270) (layer F.SilkS)
+    (fp_text reference R3 (at 0.85 -1.48 270) (layer F.SilkS)
       (effects (font (size 1 1) (thickness 0.15)))
     )
@@
       (rotate (xyz 0 0 0))
     )
+  )
+  (gr_text CANL0 (at 164.98 96.29 90) (layer F.SilkS)
+    (effects (font (size 1 1) (thickness 0.15)))
+  )
+  (gr_text GND (at 165.06 101.92 90) (layer F.SilkS)
+    (effects (font (size 1 1) (thickness 0.15)))
+  )
+  (gr_text CANH0 (at 165.01 88.73 90) (layer F.SilkS)
+    (effects (font (size 1 1) (thickness 0.15)))
+  )
+  (gr_text CANH1 (at 121.89 101.78 270) (layer F.SilkS)
+    (effects (font (size 1 1) (thickness 0.15)))
+  )
+  (gr_text CANL1 (at 121.98 95.18 270) (layer F.SilkS)
+    (effects (font (size 1 1) (thickness 0.15)))
+  )
+  (gr_text GND (at 121.9 89.55 270) (layer F.SilkS)
+    (effects (font (size 1 1) (thickness 0.15)))
   )
   (gr_text JLCJLCJLCJLC (at 174.78 96.78 90) (layer F.SilkS)
@@
   (segment (start 131.285 102.4) (end 131.33 102.355) (width 0.3048) (layer F.Cu) (net 100))
   (segment (start 130.51 102.355) (end 131.33 102.355) (width 0.3048) (layer F.Cu) (net 100))
+  (segment (start 122.58 106.975) (end 122.54 107.015) (width 0.3048) (layer F.Cu) (net 100))
   (segment (start 125.89 106.975) (end 130.51 102.355) (width 0.3048) (layer F.Cu) (net 100))
-  (segment (start 122.58 106.975) (end 122.54 107.015) (width 0.3048) (layer F.Cu) (net 100))
   (segment (start 125.89 106.975) (end 122.58 106.975) (width 0.3048) (layer F.Cu) (net 100))
   (segment (start 117.875 102.35) (end 122.54 107.015) (width 0.3048) (layer F.Cu) (net 100))
-  (segment (start 116.05 102.35) (end 117.875 102.35) (width 0.3048) (layer F.Cu) (net 100))
+  (segment (start 125.9 93.785) (end 125.9 94.41) (width 0.3048) (layer F.Cu) (net 101))
   (segment (start 125.9 94.41) (end 125.9 97.87) (width 0.3048) (layer F.Cu) (net 101))
-  (segment (start 125.9 93.785) (end 125.9 94.41) (width 0.3048) (layer F.Cu) (net 101))
+  (segment (start 125.9 97.87) (end 127.64 97.87) (width 0.3048) (layer F.Cu) (net 101))
+  (segment (start 127.64 97.87) (end 130.855 101.085) (width 0.3048) (layer F.Cu) (net 101))
+  (segment (start 125.9 97.87) (end 116.65 97.87) (width 0.3048) (layer F.Cu) (net 101))
   (segment (start 130.855 101.085) (end 131.33 101.085) (width 0.3048) (layer F.Cu) (net 101))
-  (segment (start 127.64 97.87) (end 130.855 101.085) (width 0.3048) (layer F.Cu) (net 101))
-  (segment (start 125.9 97.87) (end 127.64 97.87) (width 0.3048) (layer F.Cu) (net 101))
   (segment (start 116.65 97.87) (end 116.05 97.27) (width 0.3048) (layer F.Cu) (net 101))
-  (segment (start 125.9 97.87) (end 116.65 97.87) (width 0.3048) (layer F.Cu) (net 101))
   (segment (start 170.925 91.735) (end 170.93 91.73) (width 0.3048) (layer F.Cu) (net 102))
   (segment (start 163.365 91.73) (end 163.34 91.705) (width 0.3048) (layer F.Cu) (net 102))
@@
   (segment (start 159.77 96.79) (end 159.81 96.83) (width 0.3048) (layer F.Cu) (net 105))
   (segment (start 159.77 93.605) (end 159.77 96.79) (width 0.3048) (layer F.Cu) (net 105))
+  (segment (start 116.05 102.35) (end 117.875 102.35) (width 0.3048) (layer F.Cu) (net 100))
   (zone (net 2) (net_name VCC) (layer F.Cu) (hatch edge 0.508)
     (connect_pads (clearance 0.254))
     (min_thickness 0.254)
-    (fill yes (arc_segments 16) (thermal_gap 0.254) (thermal_bridge_width 0.508))
+    (fill (arc_segments 16) (thermal_gap 0.254) (thermal_bridge_width 0.508))
     (polygon
       (pts
@@
     (connect_pads (clearance 0.254))
     (min_thickness 0.254)
-    (fill yes (arc_segments 16) (thermal_gap 0.254) (thermal_bridge_width 0.508))
+    (fill (arc_segments 16) (thermal_gap 0.254) (thermal_bridge_width 0.508))
     (polygon
       (pts
